Commit message: fixed waypoint policy for torque control with sawyer

File: gym-bullet-extensions/gym_bullet_extensions/data/cylinder_block.urdf (robot description, URDF)
Before this commit: robot cylinder, 1 links, 0 joints
Links:
- link cylinder_base_link: mass 2.0 -> 5.0; geometry collision cylinder length=0.25 radius=0.08; visual cylinder length=0.25 radius=0.08

Commit message: changed search space and object mass

File: gym-bullet-extensions/gym_bullet_extensions/data/cylinder_block.urdf (robot description, URDF)
Before this commit: robot cylinder, 1 links, 0 joints
Links:
- link cylinder_base_link: mass 5.0 -> 10.0
